Commit message: remove useless comments

File: rotors_simulator/rotors_description/urdf/firefly.xacro (robot description, xacro)
@@ -184,53 +184,3 @@
     <xacro:insert_block name="rotor_inertia" />
   </xacro:vertical_rotor>
-<!--
-<link name="connector1">
-    <visual name="connector1_visual">
-      <origin xyz="0 0 0" rpy="0 0 0"/>
-      <geometry>
-      <box size="0.01 0.01 0.01"/>
-      </geometry>
-    </visual>
-    <inertial>
-    <mass value="0.001"/>
-    <origin xyz="0.0 0 0" rpy=" 0 0 0"/>
-    <inertia
-        ixx="0.001" ixy="0" ixz="0"
-        iyy="0.001" iyz="0"
-        izz="0.001"
-    />
-    </inertial>
-  </link>
-<joint type="revolute" name="connector1_joint">
-   <origin xyz="0.0 0 -0.05" rpy="0 0 0"/>
-   <child link="connector1"/>
-   <parent link="${namespace}/base_link"/>
-   <axis xyz="0 1 0" />
-    <limit effort="300" lower="-1.57" upper="1.57" velocity="1"/>
-</joint>
-<link name="connector2">
-    <visual name="connector2_visual">
-      <origin xyz="0 0 0" rpy="0 0 0"/>
-      <geometry>
-      <box size="0.01 0.01 0.01"/>
-      </geometry>
-    </visual>
-    <inertial>
-    <mass value="0.001"/>
-    <origin xyz="0.0 0 0" rpy=" 0 0 0"/>
-    <inertia
-        ixx="0.001" ixy="0" ixz="0"
-        iyy="0.001" iyz="0"
-        izz="0.001"
-    />
-    </inertial>
-  </link>
-<joint type="revolute" name="connector2_joint">
-   <origin xyz="0.0 0 0.001" rpy="0 0 0"/>
-   <child link="connector2"/>
-   <parent link="connector1"/>
-   <axis xyz="1 0 0" />
-    <limit effort="300" lower="-1.57" upper="1.57" velocity="1"/>
-</joint>
--->
 </robot>

Commit message: some change about controller and path

File: rotors_simulator/rotors_description/urdf/firefly.xacro (robot description, xacro)
@@ -190,5 +190,5 @@
 		<origin xyz="0 0.1 ${rotor_offset_top}" rpy="0 0 0" />
 		-->
-		<origin xyz="0.5 0.5 0.25" rpy="0 0 0" />
+		<origin xyz="0.5 0.5 0" rpy="0 0 0" />
 </joint>
 <link name="mass_piece">
